File: hardware/ch570sao9v.kicad_pcb (KiCad board)
At the start: 2 copper layers, 34.8 x 59.7 mm, 44 parts, among them J1 SAO, SW1 TS-1187A-B-A-B, SW2 TS-1187A-B-A-B, SW3 TS-1187A-B-A-B, SW4 SW_SPDT, U2 TPS54302, U3 CH572Q, U4 HX3608_BOOST, Y1 32MHz

Commit message: Update design
Parts:
- added C16: 1u, Resistor_SMD:R_0402_1005Metric, F.Cu at (209.6, 104.7)
- added C17: 100n, Resistor_SMD:R_0402_1005Metric, F.Cu at (203.5, 105.1)
- added C18: 100n, Resistor_SMD:R_0402_1005Metric, F.Cu at (201.7, 105.3)
- added R4: 33, cnhardware:R_0402_1005Metric_COMPACT, F.Cu at (203.9, 106.2)
- added R9: 33k, cnhardware:R_0402_1005Metric_COMPACT, F.Cu at (199.0, 103.1)
- added U5: ~, cnhardware:LGA-14_3x2.5mm_P0.5mm_LayoutBorder3x4y_EVEN_PADS, F.Cu at (201.6, 102.4)
- added U6: QMC6309, Package_BGA:WLP-4_0.83x0.83mm_P0.4mm, F.Cu at (209.6, 102.7)
- U1: moved to F.Cu
- moved C13 2.22 mm to (202.1, 97.3)
- moved TP2 2.18 mm to (203.6, 99.2)
- moved U3 2.18 mm to (201.8, 94.0)
- moved C1 1.95 mm to (204.3, 84.3)
- moved Y1 1.67 mm to (196.8, 94.6)
- moved R3 1.38 mm to (202.5, 84.1)
- moved U1 1.00 mm to (200.0, 82.0)
- moved L2 0.63 mm to (210.3, 94.9)
Routing:
- net D/C: track 8.46 -> 46.6 mm, vias 1 -> 6
- net BS1: track 10.9 -> 41.7 mm, vias 1 -> 6
- net IMUVC: track 0.00 -> 11.2 mm, vias 0 -> 2
- net VDD: track 80.1 -> 89.3 mm, vias 7 -> 5
- net GND: track 321.0 -> 325.5 mm, vias 54 -> 84
- net SCK: track 14.4 -> 17.6 mm, vias 1 -> 2
- net RES: track 8.31 -> 11.5 mm, vias 1 -> 2
- net SCS: track 10.1 -> 13.2 mm, vias 1 -> 2
- net VPP: track 47.5 -> 50.3 mm, vias 3 -> 4
- net MOSI: track 13.4 -> 16.1 mm, vias 1 -> 2
- net B2: track 41.6 -> 39.4 mm
- net SWCLK: track 25.0 -> 22.9 mm
- net SWD: track 29.5 -> 27.4 mm
- net B0: track 49.6 -> 47.5 mm
- net B1: track 58.9 -> 56.9 mm
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Other:
- board text added: "REV A UNTESTED"
- board text added: "ch570sao9v-revA"
- board text removed: "ch570sao9v-rev-"

Commit message: Update design
Parts:
- moved SW4 3.73 mm to (212.3, 136.5), turned to 0 degrees
- moved TP7 2.10 mm to (207.6, 131.8)
- moved TP9 2.10 mm to (193.3, 131.9)
Routing:
- net Net-(BT1-+): track 5.55 -> 7.92 mm
- net D/C: track 46.6 -> 45.4 mm
- net BS1: track 41.7 -> 40.7 mm
- net GND: vias 84 -> 94
Other:
- board text added: "GND VDD - - SWD SWC"
- board text removed: "GND VDD - - SWD SWCLK"
- board text removed: "VDD GND - - SWC SWD"

Commit message: Update to rev a
Parts:
- added D2: 1N4148, Diode_SMD:D_SOD-323, F.Cu at (214.9, 107.6)
- TP1: value MOSITP -> MOSI
- TP3: value DCTP -> SCK
- TP4: value DCTP -> DC
- TP5: value SCSTP -> SCS
- TP6: value RESTP -> RES
- moved TP7 1.09 mm to (207.6, 132.9)
- moved TP9 1.09 mm to (193.3, 133.0)
Connections:
- SW4 pad 2: +9V -> Net-(D2-A)
Routing:
- net GND: track 325.5 -> 296.2 mm, vias 94 -> 117
- net Net-(D2-A): track 0.00 -> 27.3 mm
- net +9V: track 76.5 -> 51.5 mm
- net Net-(BT1-+): track 7.92 -> 12.2 mm, vias 1 -> 2
- net B0: track 47.5 -> 45.7 mm
- net D/C: track 45.4 -> 45.8 mm, vias 6 -> 8
- net BS1: track 40.7 -> 40.9 mm, vias 6 -> 8
Other:
- board text added: "1.1mm Thick Max random parts (SOT-23, SOD-323) 1.25mm Thick Inductor Cap must be 1.25 to 1.6mm Thick PCB: 1.6mm Thick FR4 1 Oz Copper Lead-Free HASL"
- board text removed: "1.1mm Thick Max random parts (SOT-23, SOD-323) 1.25mm Thick Inductor Cap must be 1.25 to 1.6mm Thick"

Commit message: Update rev a
Parts:
- added C19: 4.7u, Capacitor_SMD:C_1206_3216Metric, F.Cu at (202.6, 108.3)
- R4: value 33 -> 10
- U5: value ~ -> LSM6DS3
- moved R9 3.73 mm to (200.5, 99.7), turned to 90 degrees
- moved R4 0.65 mm to (203.4, 105.7)
- moved C17 0.40 mm to (203.4, 104.7)
- moved C18 0.15 mm to (201.6, 105.2)
Routing:
- net GND: track 296.2 -> 301.1 mm, vias 117 -> 118
- net D/C: track 45.8 -> 42.5 mm
- net IMUVC: track 11.2 -> 14.4 mm
- net VDD: track 89.3 -> 87.7 mm

Commit message: Bump design
Parts:
- moved C15 1.36 mm to (191.1, 84.8), turned to 120 degrees
- moved R3 0.99 mm to (202.0, 85.0), turned to 90 degrees
- moved C1 0.31 mm to (204.4, 84.7)
- moved U1 0.15 mm to (200.0, 82.2)
Routing:
- net GND: track 301.1 -> 306.8 mm
- net VDD: track 87.7 -> 88.7 mm
- net Net-(U1-IREF): track 2.10 -> 2.65 mm
Other:
- board text added: "REV B UNTESTED"
- board text added: "VDD GND - - SWC SWD"
- board text added: "ch570sao9v-revB"
- board text removed: "GND VDD - - SWD SWC"
- board text removed: "REV A UNTESTED"
- board text removed: "ch570sao9v-revA"
